File: machine.kicad_sch (KiCad schematic)
At the start: 30 parts, among them J1 TMC2209 Y, J10 SD Card, J11 Stop, J12 Serial, J13 STM32DevV1-VCC, J14 STM32DevV1-3.3, J2 TMC2209 B, J3 X Motor, J4 Y Motor, J5 24V, J6 Buttons, J7 X limit, J8 Y limit, J9 Display, U2 K7805W-500R3

Commit message: Add stability
Parts:
- removed J11: Stop, CONN_B6B-XH-A_JST, symbol JST-XH-6A:B6B-XH-A
- removed J6: Buttons, CONN_B5B-XH-A_JST, symbol JST-XH-5A:B5B-XH-A
- added C6, C7, C8, C9: 0.1μF, symbol Device:C
- added J11: Stop, CONN_B4B-XH-A_JST, symbol JST-XH-4A:B4B-XH-A
- added J6: Hold, CONN_B2B-XH-A_JST, symbol JST-XH-2A:B2B-XH-A
- added JP1, JP2, JP3, JP4: ~, Jumper:SolderJumper-2_P1.3mm_Bridged_RoundedPad1.0x1.5mm, symbol Jumper:SolderJumper_2_Bridged
- added JP5: ~, Jumper:SolderJumper-2_P1.3mm_Open_RoundedPad1.0x1.5mm, symbol Jumper:SolderJumper_2_Open
- added R10, R9: 100, symbol Device:R
- added R11, R12: R, symbol Device:R
- added R13, R14, R15, R16: 10, symbol Device:R
- added SW1: Hold, symbol Switch:SW_Push
- added SW2: Run, symbol Switch:SW_Push
- added SW3: M1, symbol Switch:SW_Push
- added SW4: M2, symbol Switch:SW_Push
- added U1: SN74LV125ADR, SN74LV125ADR:SOIC127P600X175-14N, symbol SN74LV125:SN74LV125ADR
- R1, R2, R3, R4: value 47k -> 1k
- R8: value 3.3k -> 590
Connections:
- net +5V: now also U1.1 (1~OE), U1.10 (3~OE), U1.4 (2~OE)
- net 3.3V: now also R13.2, R14.2, R15.2, R16.2, U1.14 (VCC)
- net DIRX: now also JP3.1 (A); no longer J13.12
- net ENX: now also JP1.1 (A); no longer J13.11
- net GND: now also C6.2, C7.2, C8.2, C9.2, J11.1, J6.1, U1.7 (GND)
- net GPIO13: now also JP2.2 (B); no longer J1.7
- net GPIO15: now also J11.4, U1.8 (3Y), U1.9 (3A)
- net GPIO2: now also J11.3, U1.5 (2A), U1.6 (2Y)
- net GPIO34: now also R10.2; no longer R2.2
- net GPIO35: now also R9.2; no longer R1.2
- net GPIO36: now also R12.2; no longer R4.2
- net GPIO39: now also R11.2; no longer R3.2
- net GPIO4: now also J11.2, U1.2 (1A), U1.3 (1Y)
- net PDN (RX): now reaches J1.5
- net PDN (RX): now also JP5.1 (A)
- removed net GPIO16: J1.4, J14.10, R5.2
- net GPIO17 renamed GPIO16 (RXD)
- net GPIO16 (RXD): now also J14.10, JP4.2 (B); no longer J14.9
- new net: R16.1, SW4.2
- new net: R13.1, SW1.2
- new net: R15.1, SW3.2
- new net: R14.1, SW2.2
- new net GPIO12: J13.12, JP3.2 (B)
- new net GPIO14: J13.11, JP1.2 (B)
- new net GPIO17 (TXD): J14.9, JP5.2 (B), R5.2
- new net Hold: C6.1, J6.2, R1.2, R9.1, SW1.1
- new net M1: C8.1, R11.1, R3.2, SW3.1
- new net M2: C9.1, R12.1, R4.2, SW4.1
- new net PDN (TX): J1.4, JP4.1 (A)
- new net Run: C7.1, R10.1, R2.2, SW2.1
- new net STEPX: J1.7, JP2.1 (A)
- no-connect marks 2 -> 4
Other:
- moved on the sheet: C1, C2, C3, C4, C5, D1, J1, J10, J12, J13, J14, J2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

Commit message: Migration init
Parts:
- removed C1: 10μF, Capacitor_Tantalum_SMD:CP_EIA-6032-28_Kemet-C_Pad2.25x2.35mm_HandSolder, symbol Device:C_Polarized
- removed C2, C3: 22μF, Capacitor_Tantalum_SMD:CP_EIA-3528-21_Kemet-B_Pad1.50x2.35mm_HandSolder, symbol Device:C_Polarized
- removed D1: LED, LED_THT:LED_Rectangular_W3.9mm_H1.9mm, symbol Device:LED
- removed J1: TMC2209 Y, CONN8_LFBN-RC_SUL, symbol HDR-08POS:PPPC081LFBN-RC
- removed J2: TMC2209 B, CONN8_LFBN-RC_SUL, symbol HDR-08POS:PPPC081LFBN-RC
- removed J3: X Motor, CONN_B4B-XH-A_JST, symbol JST-XH-4A:B4B-XH-A
- removed J4: Y Motor, CONN_B4B-XH-A_JST, symbol JST-XH-4A:B4B-XH-A
- removed J5: 24V, CONN_B2B-XH-A_JST, symbol JST-XH-2A:B2B-XH-A
- removed JP1, JP2, JP3, JP4: ~, Jumper:SolderJumper-2_P1.3mm_Bridged_RoundedPad1.0x1.5mm, symbol Jumper:SolderJumper_2_Bridged
- removed JP5: ~, Jumper:SolderJumper-2_P1.3mm_Open_RoundedPad1.0x1.5mm, symbol Jumper:SolderJumper_2_Open
- removed L1: 15μH, Inductor_SMD:L_SXN_SMDRI74, symbol Device:L_Ferrite
- removed R5: 1k, Resistor_SMD:R_0805_2012Metric_Pad1.20x1.40mm_HandSolder, symbol Device:R
- removed R8: 590, Resistor_SMD:R_0805_2012Metric_Pad1.20x1.40mm_HandSolder, symbol Device:R
- removed U2: K7805W-500R3, Package_TO_SOT_THT:TO-220-3_Vertical, symbol Regulator_Linear:LM7805_TO220
- added J15: Conn_01x04_Socket, symbol Connector:Conn_01x04_Socket
- added J16: Conn_01x06_Socket, symbol Connector:Conn_01x06_Socket
Connections:
- net DIRY renamed GPIO26_Y_DIR
- net ENY renamed GPIO27_Y_EN
- net GPIO12: no longer names the net of J13.12
- net GPIO13: no longer names the net of J13.13
- net GPIO14: no longer names the net of J13.11
- net GPIO16 (RXD): no longer names the net of J14.10
- net GPIO17 (TXD): no longer names the net of J14.9
- net GPIO25 renamed GPIO25_Y_STEP
Other:
- added sheet IO (IO.kicad_sch)
- added sheet MCU (MCU.kicad_sch)
- added sheet Power (power.kicad_sch)

Commit message: Transformation in progress
Parts:
- removed C4, C5: 4.7nF, Capacitor_SMD:C_0805_2012Metric_Pad1.18x1.45mm_HandSolder, symbol Device:C
- removed C6, C7, C8, C9: 0.1μF, symbol Device:C
- removed J10: SD Card, CONN_B6B-XH-A_JST, symbol JST-XH-6A:B6B-XH-A
- removed J11: Stop, CONN_B4B-XH-A_JST, symbol JST-XH-4A:B4B-XH-A
- removed J12: Serial, Connector_PinSocket_2.54mm:PinSocket_1x03_P2.54mm_Vertical, symbol Connector:Conn_01x03_Pin
- removed J13: STM32DevV1-VCC, CONN15_PPPC151LFBN-RC_SUL, symbol HDR-15POS:PPPC151LFBN-RC
- removed J14: STM32DevV1-3.3, CONN15_PPPC151LFBN-RC_SUL, symbol HDR-15POS:PPPC151LFBN-RC
- removed J15: Conn_01x04_Socket, symbol Connector:Conn_01x04_Socket
- removed J16: Conn_01x06_Socket, symbol Connector:Conn_01x06_Socket
- removed J6: Hold, CONN_B2B-XH-A_JST, symbol JST-XH-2A:B2B-XH-A
- removed J7: X limit, CONN_B3B-XH-A_JST, symbol JST-XH-3A:B3B-XH-A
- removed J8: Y limit, CONN_B3B-XH-A_JST, symbol JST-XH-3A:B3B-XH-A
- removed J9: Display, CONN_B4B-XH-A_JST, symbol JST-XH-4A:B4B-XH-A
- removed R1, R2, R3, R4: 1k, Resistor_SMD:R_0805_2012Metric_Pad1.20x1.40mm_HandSolder, symbol Device:R
- removed R10, R9: 100, symbol Device:R
- removed R11, R12: R, symbol Device:R
- removed R13, R14, R15, R16: 10, symbol Device:R
- removed R6: 200, Resistor_SMD:R_0805_2012Metric_Pad1.20x1.40mm_HandSolder, symbol Device:R
- removed R7: 1.2k, Resistor_SMD:R_0805_2012Metric_Pad1.20x1.40mm_HandSolder, symbol Device:R
- removed SW1: Hold, symbol Switch:SW_Push
- removed SW2: Run, symbol Switch:SW_Push
- removed SW3: M1, symbol Switch:SW_Push
- removed SW4: M2, symbol Switch:SW_Push
- removed U1: SN74LV125ADR, SN74LV125ADR:SOIC127P600X175-14N, symbol SN74LV125:SN74LV125ADR
Connections:
- no-connect marks 4 -> 0
