File: MCU.kicad_sch (KiCad schematic)
At the start: 0 parts

Commit message: Transformation in progress
Parts:
- added C14: 22μF, Capacitor_SMD:C_0805_2012Metric_Pad1.18x1.45mm_HandSolder, symbol Device:C
- added C15, C16, C17, C18: 100nF, Capacitor_SMD:C_0805_2012Metric_Pad1.18x1.45mm_HandSolder, symbol Device:C
- added C19: 10μF, Capacitor_SMD:C_0805_2012Metric_Pad1.18x1.45mm_HandSolder, symbol Device:C
- added D8: SP0503BAHTG, SP0503BAHTG:SOT143, symbol SP0503BAHTG:SP0503BAHTG
- added D9: B340A-13-F, Diode_SMD:D_SMC, symbol Diode:B340
- added J15: Display, Connector_PinHeader_2.54mm:PinHeader_1x04_P2.54mm_Vertical, symbol Connector:Conn_01x04_Socket
- added J18: MEM2061-01-188-00-A_REVA, MEM2061-01-188-00-A_REVA:GCT_MEM2061-01-188-00-A_REVA, symbol MEM2061_01_188_00_A:MEM2061-01-188-00-A_REVA
- added J19: TYPE-C 15PIN, 10155435-00011LF:AMPHENOL_10155435-00011LF, symbol 10155435_00011LF:10155435-00011LF
- added Q1, Q2: PMBT6428,215, symbol Simulation_SPICE:NPN
- added R25, R26, R29, R30: 10k, Resistor_SMD:R_0805_2012Metric_Pad1.20x1.40mm_HandSolder, symbol Device:R
- added R27, R28: 1k, Resistor_SMD:R_0805_2012Metric_Pad1.20x1.40mm_HandSolder, symbol Device:R
- added R31, R32: 5.1k, Resistor_SMD:R_0805_2012Metric_Pad1.20x1.40mm_HandSolder, symbol Device:R
- added R33: 22.1k, Resistor_SMD:R_0805_2012Metric_Pad1.20x1.40mm_HandSolder, symbol Device:R
- added R34: 47.5k, Resistor_SMD:R_0805_2012Metric_Pad1.20x1.40mm_HandSolder, symbol Device:R
- added R35: 2k, Resistor_SMD:R_0805_2012Metric_Pad1.20x1.40mm_HandSolder, symbol Device:R
- added R36, R37: 0, Resistor_SMD:R_0805_2012Metric_Pad1.20x1.40mm_HandSolder, symbol Device:R
- added SW5: Reset, Button_Switch_SMD:SW_Push_SPST_NO_Alps_SKRK, symbol Switch:SW_Push
- added SW6: Boot, Button_Switch_SMD:SW_Push_SPST_NO_Alps_SKRK, symbol Switch:SW_Push
- added TP1: ~, TestPoint:TestPoint_Pad_D1.0mm, symbol Connector:TestPoint
- added U5: ESP32-WROOM-32E 4MB, ESP32-WROOM-32E-N4:ESP32-WROOM-32E_EXP, symbol ESP32-WROOM-32E-N4:ESP32-WROOM-32E_4MB
- added U6: CP2102-GMR, INTERFACE-CP2102-GMR_QFN28_:QFN28G_0.5-5X5MM, symbol CP2102_GMR:INTERFACE-CP2102-GMR_QFN28_
Connections:
- new net: Q1.2 (B), R25.1
- new net: R27.1, SW5.1
- new net: Q2.2 (B), R26.1
- new net: R36.1, U6.25 (RXD)
- new net: R37.1, U6.26 (TXD)
- new net: R33.1, R34.2, U6.8 (VBUS)
- new net: R35.2, U6.9 (~{RST})
- new net: J19.A5 (CC1), R32.1
- new net: J19.B5 (CC2), R31.2
- new net: R28.1, SW6.1
- new net +3V3: C14.2, C15.2, C16.2, C18.2, C19.2, J18.4 (VDD), R29.1, R30.2, R35.1, U5.2 (3V3), U6.6 (VDD), U6.7 (REGIN)
- new net +5V: D9.1 (K)
- new net 3.3V: J15.2 (Pin_2)
- new net D+: D8.2, J19.A6 (DP1), J19.B6 (DP2), U6.4 (D+)
- new net D-: D8.3, J19.A7 (DN1), J19.B7 (DN2), U6.5 (D-)
- new net DTR: Q2.3 (E), R25.2, U6.28 (DTR)
- new net D_SCK: J15.3 (Pin_3), U5.24 (IO2)
- new net D_SDA: J15.4 (Pin_4), U5.23 (IO15)
- new net ESP_EN: C17.1, Q1.1 (C), R29.2, SW5.2, U5.3 (EN)
- new net GND: C14.1, C15.1, C16.1, C17.2, C18.1, C19.1, D8.1, J15.1 (Pin_1), J18.10 (CD2), J18.11 (GND), J18.12 (GND__1), J18.6 (VSS), J19.A1_B12 (GND), J19.B1_A12 (GND__1), J19.SH1 (SHIELD), J19.SH2 (SHIELD__1), J19.SH3 (SHIELD__2), J19.SH4 (SHIELD__3), R27.2, R28.2, R31.1, R32.2, R34.1, U5.1 (GND), U5.15 (GND), U5.38 (GND), U5.39 (GND), U5.40 (GND), U5.41 (GND), U5.42 (GND), U5.43 (GND), U5.44 (GND), U5.45 (GND), U5.46 (GND), U5.47 (GND), U6.29 (GND@1), U6.3 (GND)
- new net GPIO34: U5.6 (IO34)
- new net GPIO35: U5.7 (IO35)
- new net GPIO36: U5.4 (SENSOR_VP)
- new net GPIO39: U5.5 (SENSOR_VN)
- new net GPIO_0: Q2.1 (C), R30.1, SW6.2, U5.25 (IO0)
- new net I2S_BCK: U5.36 (IO22)
- new net I2S_DATA: U5.33 (IO21)
- new net I2S_WS: U5.26 (IO4)
- new net RTS: Q1.3 (E), R26.2, U6.24 (RTS)
- new net RXD0: R37.2, U5.34 (RXD0)
- new net SD_CS: J18.2 (CD/DAT3), U5.29 (IO5)
- new net SD_MISO: J18.7 (DAT0), U5.31 (IO19)
- new net SD_MOSI: J18.3 (CMD), U5.37 (IO23)
- new net SD_SCK: J18.5 (CLK), U5.30 (IO18)
- new net TXD0: R36.2, U5.35 (TXD0)
- new net VBUS: D8.4, D9.2 (A), J19.A4_B9 (VBUS), J19.B4_A9 (VBUS__1), R33.2, TP1.1
- new net X_RXD: U5.27 (IO16)
- new net X_TXD: U5.28 (IO17)
- no-connect marks 0 -> 22

Commit message: Finalization v2.0
Parts:
- removed C16: 100nF, Capacitor_SMD:C_0805_2012Metric_Pad1.18x1.45mm_HandSolder, symbol Device:C
- removed J15: Display, Connector_PinHeader_2.54mm:PinHeader_1x04_P2.54mm_Vertical, symbol Connector:Conn_01x04_Socket
- removed J18: MEM2061-01-188-00-A_REVA, MEM2061-01-188-00-A_REVA:GCT_MEM2061-01-188-00-A_REVA, symbol MEM2061_01_188_00_A:MEM2061-01-188-00-A_REVA
- removed Q1, Q2: PMBT6428,215, symbol Simulation_SPICE:NPN
- removed R37: 0, Resistor_SMD:R_0805_2012Metric_Pad1.20x1.40mm_HandSolder, symbol Device:R
- added Q1, Q2: SS8050, Package_TO_SOT_SMD:SOT-23, symbol Transistor_BJT:SS8050
- added R12: 0, Resistor_SMD:R_0805_2012Metric_Pad1.20x1.40mm_HandSolder, symbol Device:R
- J7: renamed from J19; footprint 10155435-00011LF:AMPHENOL_10155435-00011LF -> 10155435_00011LF:AMPHENOL_10155435-00011LF
- U4: renamed from U6; footprint INTERFACE-CP2102-GMR_QFN28_:QFN28G_0.5-5X5MM -> CP2102_GMR:QFN28G_0.5-5X5MM
- renumbered C19 to C10, C15 to C11, C14 to C12, C17 to C8, C18 to C9, D9 to D8, D8 to D9, R25 to R11, R36 to R13, R26 to R14, R32 to R15, R31 to R16, R27 to R17, R29 to R18, R30 to R19, R28 to R20, R33 to R21, R35 to R22, R34 to R23, SW5 to SW1, SW6 to SW2
Connections:
- net DTR: now also Q2.2 (E)
- net ESP_EN: now also Q1.3 (C)
- net RTS: now also Q1.2 (E)
- net RXD0: now also R12.1
- net TXD0: now also R13.1; no longer R13.2
- net at R11.1: now also Q1.1 (B)
- net at R14.1: now also Q2.1 (B)
- net at U4.25 (RXD): now also R13.2; no longer R13.1
- net at U4.26 (TXD): now also R12.2
- net LED_HOLD: now reaches U5.10 (IO25)
- net LED_RUN: now reaches U5.11 (IO26)
- net LED_ALARM: now reaches U5.12 (IO27)
- net X_POS_LIM: now reaches U5.16 (IO13)
- net Y_ALL_LIM: now reaches U5.8 (IO32)
- net X_NEG_LIM: now reaches U5.9 (IO33)
- net GPIO34 renamed BTN_RUN
- net GPIO35 renamed BTN_HOLD
- net GPIO36 renamed BTN_M1
- net GPIO39 renamed BTN_M2
- net GPIO_0 renamed GPIO0
- net GPIO0: now also Q2.3 (C)
- no-connect marks 22 -> 21
Other:
- moved on the sheet: C10, C11, C12, C8, C9, D8, D9, J7, R11, R13, R14, R15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
