File: power.kicad_sch (KiCad schematic)
At the start: 34 parts, among them J1 TMC2209 Y, J17 SW, J2 TMC2209 B, J3 X Motor, J4 Y Motor, J5 24V, K1 ZGT-40DD, U2 K7805W-500R3, U3 NCP1117IST33T3G, U4 74AHCT595

Commit message: Transformation in progress
Parts:
- added D2, D3, D4, D5, D6, D7: LED, LED_SMD:LED_0603_1608Metric, symbol Device:LED
- added R19, R20, R21, R22, R23, R24: 10k, Resistor_SMD:R_0805_2012Metric_Pad1.20x1.40mm_HandSolder, symbol Device:R
- J1, J2: footprint CONN8_LFBN-RC_SUL -> HDR-08POS:CONN8_LFBN-RC_SUL
- J17: value SW -> PWR SW; footprint CONN_B2B-XH-A_JST -> JST-XH-2A:CONN_B2B-XH-A_JST
- J3, J4: footprint CONN_B4B-XH-A_JST -> JST-XH-4A:CONN_B4B-XH-A_JST
- J5: value 24V -> PWR IN; footprint CONN_B2B-XH-A_JST -> JST-XH-2A:CONN_B2B-XH-A_JST
- U3: footprint SOT-223_NCP1117IST33T3G_OSI -> NCP1117IST33T3G:SOT-223_NCP1117IST33T3G_OSI
- U4: footprint (none) -> Package_SO:TSSOP-16_4.4x5mm_P0.65mm
Connections:
- net DIRY is gone; now on net Y_DIR: J4.3
- net ENY is gone; now on net Y_ENABLE: J4.2
- net STEPY is gone; now on net Y_STEP: J4.4
- net +3V3: now also U3.4 (Tab)
- net GND: now also D2.1 (K), D3.1 (K), D4.1 (K), D5.1 (K), D6.1 (K), D7.1 (K)
- net X_DIR: now also R20.1
- net X_ENABLE: now also R19.1
- net X_STEP: now also R21.1
- net Y_DIR: now also R23.2
- net Y_ENABLE: now also R24.2
- net Y_STEP: now also R22.2
- net GPIO16 (RXD) renamed X_RXD
- net GPIO17 (TXD) renamed X_TXD
- new net: D4.2 (A), R21.2
- new net: D5.2 (A), R22.1
- new net: D3.2 (A), R20.2
- new net: D2.2 (A), R19.2
- new net: D7.2 (A), R24.1
- new net: D6.2 (A), R23.1
- no-connect marks 4 -> 3
Other:
- moved on the sheet: C12, C13, H1, H2, H3, H4, H5, H6, J1, J2, J3, J4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

Commit message: Finalization v2.0
Parts:
- removed J17: PWR SW, JST-XH-2A:CONN_B2B-XH-A_JST, symbol JST-XH-2A:B2B-XH-A
- removed JP1, JP2: ~, Jumper:SolderJumper-2_P1.3mm_Bridged_RoundedPad1.0x1.5mm, symbol Jumper:SolderJumper_2_Bridged
- added J2: Y Motor PWR, Connector_Phoenix_MSTB:PhoenixContact_MSTBVA_2,5_2-G-5,08_1x02_P5.08mm_Vertical, symbol JST-XH-2A:B2B-XH-A
- added JP4: MS1, Jumper:SolderJumper-2_P1.3mm_Bridged_RoundedPad1.0x1.5mm, symbol Jumper:SolderJumper_2_Bridged
- added JP5: MS2, Jumper:SolderJumper-2_P1.3mm_Bridged_RoundedPad1.0x1.5mm, symbol Jumper:SolderJumper_2_Bridged
- C1: footprint Capacitor_Tantalum_SMD:CP_EIA-6032-28_Kemet-C_Pad2.25x2.35mm_HandSolder -> Capacitor_Tantalum_SMD:CP_EIA-6032-28_Kemet-C_HandSolder
- C2, C3: footprint Capacitor_Tantalum_SMD:CP_EIA-3528-21_Kemet-B_Pad1.50x2.35mm_HandSolder -> Capacitor_Tantalum_SMD:CP_EIA-3528-21_Kemet-B_HandSolder
- C4: renamed from C10; footprint Capacitor_Tantalum_SMD:CP_EIA-6032-28_Kemet-C_Pad2.25x2.35mm_HandSolder -> Capacitor_Tantalum_SMD:CP_EIA-6032-28_Kemet-C_HandSolder
- C5: renamed from C11; footprint Capacitor_Tantalum_SMD:CP_EIA-6032-28_Kemet-C_Pad2.25x2.35mm_HandSolder -> Capacitor_Tantalum_SMD:CP_EIA-6032-28_Kemet-C_HandSolder
- H1, H2, H3, H4, H5, H6: footprint (none) -> MountingHole:MountingHole_3.2mm_M3_DIN965_Pad
- J1: renamed from J5; footprint JST-XH-2A:CONN_B2B-XH-A_JST -> Connector_Phoenix_MSTB:PhoenixContact_MSTBVA_2,5_2-G-5,08_1x02_P5.08mm_Vertical
- J6: renamed from J4; value Y Motor -> Y Motor Control
- JP1: renamed from JP4; value ~ -> PDN
- JP2: renamed from JP5; value ~ -> PDN
- JP3: value ~ -> CK
- renumbered C12 to C6, C13 to C7, J1 to J3, J2 to J4, J3 to J5, R8 to R1, R24 to R10, R19 to R2, R20 to R3, R21 to R4, R18 to R5, R5 to R6, R17 to R7, R22 to R8, R23 to R9, U2 to U1, U3 to U2, U4 to U3
Connections:
- net ENX is gone; now on net X_ENABLE: J3.1
- net STEPX is gone; now on net X_STEP: J3.7
- net 24V: now also J2.2
- net GND: now also JP3.2 (B), J2.1, JP4.2 (B), JP5.2 (B); no longer J3.2, J3.3, J3.6
- net X_DIR: now also J3.8; no longer JP3.2 (B)
- net PWR SW: now reaches K1.3 (3+)
- net DIRX renamed CK
- net CK: now also J3.6; no longer J3.8
- net I2S_MR#: no longer names the net of C7.2, R5.1, U3.10 (~{SRCLR})
- new net MS1: J3.2, JP4.1 (A)
- new net MS2: J3.3, JP5.1 (A)
Other:
- note added: "DIR"
- note added: "ENABLE"
- note added: "GND"
- note added: "STEP"
- note added: "VDD"
- note added: "VM"
- moved on the sheet: C7, H1, H2, H3, H4, H5, H6, J1, K1, R5, R7
